File: study focus device/buttons1.kicad_sch (KiCad schematic)
At the start: 17 parts, among them U1 MCP23017_SP

Commit message: More additions to the circuit
Parts:
- renumbered S to S81
Changed lines of the file:
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@@
 		(on_board yes)
 		(dnp no)
-		(property "Reference" "S"
+		(property "Reference" "S?"
 			(at 158.75 71.628 0)
 			(effects
@@
 				(path "/33a9b268-fa43-451b-98e7-c69879a56f92/59c9e324-f072-4507-a391-6a085bfc55dd"
 					(reference "S81")
+					(unit 1)
+				)
+				(path "/33a9b268-fa43-451b-98e7-c69879a56f92/7f0f166a-8b8a-48ce-8614-d2f44b93b1ca"
+					(reference "S?")
 					(unit 1)
 				)
@@
 		(dnp no)
 		(fields_autoplaced yes)
-		(property "Reference" "#PWR"
+		(property "Reference" "#PWR?"
 			(at 116.84 95.25 0)
 			(effects
@@
 				(path "/33a9b268-fa43-451b-98e7-c69879a56f92/59c9e324-f072-4507-a391-6a085bfc55dd"
 					(reference "#PWR096")
+					(unit 1)
+				)
+				(path "/33a9b268-fa43-451b-98e7-c69879a56f92/7f0f166a-8b8a-48ce-8614-d2f44b93b1ca"
+					(reference "#PWR?")
 					(unit 1)
 				)
@@
 		(dnp no)
 		(fields_autoplaced yes)
-		(property "Reference" "#PWR"
+		(property "Reference" "#PWR?"
 			(at 171.45 72.39 0)
 			(effects
@@
 					(unit 1)
 				)
+				(path "/33a9b268-fa43-451b-98e7-c69879a56f92/7f0f166a-8b8a-48ce-8614-d2f44b93b1ca"
+					(reference "#PWR?")
+					(unit 1)
+				)

Commit message: more work
Parts:
- added C1: C, Capacitor_THT:C_Radial_D5.0mm_H11.0mm_P2.00mm, symbol Device:C
- renumbered S81 to S?, S15 to S?, S13 to S?, S8 to S?, S6 to S?, S10 to S?, S12 to S?, S7 to S?, S11 to S?, S14 to S?, S5 to S?, S4 to S?, S16 to S?, S3 to S?, S9 to S?, S2 to S?, U1 to U?
Connections:
- net +3V3: now also C1.1
- net GND: now also C1.2
Other:
- moved on the sheet: S?
