File: study focus device/leds.kicad_sch (KiCad schematic)
At the start: 65 parts, among them U7 MAX7219

Commit message: more changes to the pcb
Connections:
- net +5V: now reaches U7.19 (V+)
Changed lines of the file:
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@@
+	(wire
+		(pts
+			(xy 39.37 24.13) (xy 39.37 27.94)
+		)
+		(stroke
+			(width 0)
+			(type default)
+		)
+	)
 	(wire
 		(pts
@@
 					(unit 1)
 				)
+			)
+		)
+	)
+	(symbol
+		(lib_id "power:+5V")
+		(at 39.37 24.13 0)
+		(unit 1)
+		(exclude_from_sim no)
+		(in_bom yes)
+		(on_board yes)
+		(dnp no)
+		(fields_autoplaced yes)
+		(property "Reference" "#PWR0133"
+			(at 39.37 27.94 0)
+			(effects
+				(font
+					(size 1.27 1.27)
+				)
+				(hide yes)
+			)
+		)
+		(property "Value" "+5V"
+			(at 39.37 19.05 0)
+			(effects
+				(font
+					(size 1.27 1.27)
+				)
+			)
+		)
+		(property "Footprint" ""
+			(at 39.37 24.13 0)
+			(effects
+				(font
+					(size 1.27 1.27)
+				)
+				(hide yes)
+			)
+		)
+		(property "Datasheet" ""
+			(at 39.37 24.13 0)
+			(effects
+				(font
+					(size 1.27 1.27)
+				)
+				(hide yes)
+			)
+		)
+		(property "Description" "Power symbol creates a global label with name \"+5V\""
+			(at 39.37 24.13 0)
+			(effects
+				(font
+					(size 1.27 1.27)
+				)
+				(hide yes)
+			)
+		)
+		(pin "1"
+		)
+		(instances
+			(project ""
+				(path "/33a9b268-fa43-451b-98e7-c69879a56f92/03c5c2bd-4970-4d56-a43f-707c6428028e"
+					(reference "#PWR0133")
+					(unit 1)
+				)

Commit message: more work
Parts:
- added C2: C, Capacitor_THT:C_Radial_D5.0mm_H11.0mm_P2.00mm, symbol Device:C
- renumbered D31 to D?, D39 to D?, D46 to D?, D12 to D?, D3 to D?, D1 to D?, D29 to D?, D15 to D?, D20 to D?, D22 to D?, D57 to D?, D54 to D?, D49 to D?, D43 to D?, D38 to D?, D50 to D?, D37 to D?, D26 to D?, D5 to D?, D56 to D?, D55 to D?, D19 to D?, D53 to D?, D6 to D?, D21 to D?, D14 to D?, D11 to D?, D47 to D?, D34 to D?, D58 to D?, D9 to D?, D51 to D?, D63 to D?, D45 to D?, D64 to D?, D59 to D?, D10 to D?, D27 to D?, D42 to D?, D40 to D?, D13 to D?, D2 to D?, D4 to D?, D36 to D?, D61 to D?, D16 to D?, D52 to D?, D62 to D?, D48 to D?, D17 to D?, D32 to D?, D8 to D?, D23 to D?, D25 to D?, D28 to D?, D30 to D?, D33 to D?, D44 to D?, D7 to D?, D18 to D?, D41 to D?, D35 to D?, D24 to D?, D60 to D?, U7 to U?
Connections:
- net +5V: now also C2.1
- net GND: now also C2.2
