File: study focus device/leds2.kicad_sch (KiCad schematic)
At the start: 33 parts, among them U8 MAX7219

Commit message: more changes to the pcb
Connections:
- net +5V: now reaches U8.19 (V+)
Changed lines of the file:
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@@
+	(wire
+		(pts
+			(xy 57.15 52.07) (xy 57.15 57.15)
+		)
+		(stroke
+			(width 0)
+			(type default)
+		)
+	)
 	(wire
 		(pts
@@
 					(unit 1)
 				)
+			)
+		)
+	)
+	(symbol
+		(lib_id "power:+5V")
+		(at 57.15 52.07 0)
+		(unit 1)
+		(exclude_from_sim no)
+		(in_bom yes)
+		(on_board yes)
+		(dnp no)
+		(fields_autoplaced yes)
+		(property "Reference" "#PWR0134"
+			(at 57.15 55.88 0)
+			(effects
+				(font
+					(size 1.27 1.27)
+				)
+				(hide yes)
+			)
+		)
+		(property "Value" "+5V"
+			(at 57.15 46.99 0)
+			(effects
+				(font
+					(size 1.27 1.27)
+				)
+			)
+		)
+		(property "Footprint" ""
+			(at 57.15 52.07 0)
+			(effects
+				(font
+					(size 1.27 1.27)
+				)
+				(hide yes)
+			)
+		)
+		(property "Datasheet" ""
+			(at 57.15 52.07 0)
+			(effects
+				(font
+					(size 1.27 1.27)
+				)
+				(hide yes)
+			)
+		)
+		(property "Description" "Power symbol creates a global label with name \"+5V\""
+			(at 57.15 52.07 0)
+			(effects
+				(font
+					(size 1.27 1.27)
+				)
+				(hide yes)
+			)
+		)
+		(pin "1"
+		)
+		(instances
+			(project ""
+				(path "/33a9b268-fa43-451b-98e7-c69879a56f92/3da0d8d2-ae8f-4a31-9bd3-b64bfa5d9d1f"
+					(reference "#PWR0134")
+					(unit 1)
+				)

Commit message: more work
Parts:
- added C3: C, Capacitor_THT:C_Radial_D5.0mm_H11.0mm_P2.00mm, symbol Device:C
- renumbered D77 to D?, D96 to D?, D73 to D?, D95 to D?, D94 to D?, D91 to D?, D92 to D?, D66 to D?, D83 to D?, D65 to D?, D85 to D?, D78 to D?, D69 to D?, D75 to D?, D81 to D?, D90 to D?, D70 to D?, D82 to D?, D71 to D?, D89 to D?, D80 to D?, D72 to D?, D84 to D?, D93 to D?, D86 to D?, D76 to D?, D87 to D?, D67 to D?, D79 to D?, D88 to D?, D74 to D?, D68 to D?, U8 to U?
Connections:
- net +5V: now also C3.1
- net GND: now also C3.2
