File: study focus device/study focus device.kicad_sch (KiCad schematic)
At the start: 1 part, among them U1 MCP23017_SP

Commit message: more additions
Parts:
- removed U1: MCP23017_SP, Package_DIP:DIP-28_W7.62mm, symbol Interface_Expansion:MCP23017_SP
Other:
- added sheet 16 Buttons (buttons1.kicad_sch)
- added sheet 16 Buttons1 (buttons1.kicad_sch)
- added sheet 16 Buttons2 (buttons1.kicad_sch)
- added sheet 16 Buttons3 (buttons1.kicad_sch)
- added sheet 16 Buttons4 (buttons1.kicad_sch)
- added sheet 16 Buttons5 (buttons1.kicad_sch)

Commit message: More additions to the circuit
Other:
- added sheet LEDS (leds.kicad_sch)
- added sheet LEDS2 (leds2.kicad_sch)
Changed lines of the file:
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@@
+	(wire
+		(pts
+			(xy 63.5 172.72) (xy 64.77 172.72)
+		)
+		(stroke
+			(width 0)
+			(type default)
+		)
+	)
 	(wire
 		(pts
@@
 	(wire
 		(pts
+			(xy 63.5 181.61) (xy 64.77 181.61)
+		)
+		(stroke
+			(width 0)
+			(type default)
+		)
+	)
+	(wire
+		(pts
 			(xy 67.31 85.09) (xy 71.12 85.09)
 		)
@@
 		(pts
 			(xy 67.31 68.58) (xy 71.12 68.58)
+		)
+		(stroke
+			(width 0)
+			(type default)
+		)
+	)
+	(wire
+		(pts
+			(xy 64.77 172.72) (xy 64.77 181.61)
 		)
 		(stroke
@@
 				)
 			)
+		)
+	)
+	(sheet
+		(at 17.78 154.94)
+		(size 45.72 19.05)
+		(exclude_from_sim no)
+		(in_bom yes)
+		(on_board yes)
+		(dnp no)
+		(fields_autoplaced yes)
+		(stroke
+			(width 0.1524)
+			(type solid)
+		)
+		(fill
+			(color 0 0 0 0.0000)
+		)
+		(property "Sheetname" "LEDS"
+			(at 17.78 154.2284 0)
+			(effects
+				(font
+					(size 1.27 1.27)
+				)
+				(justify left bottom)
+			)
+		)
+		(property "Sheetfile" "leds.kicad_sch"
+			(at 17.78 174.5746 0)
+			(effects
+				(font
+					(size 1.27 1.27)
+				)
+				(justify left top)
+			)
+		)
+		(pin "CLK" bidirectional
+			(at 63.5 157.48 0)
+			(effects
+				(font
+					(size 1.27 1.27)
+				)
+				(justify right)
+			)
+		)
+		(pin "DIN" input
+			(at 63.5 160.02 0)
+			(effects
+				(font
+					(size 1.27 1.27)
+				)
+				(justify right)
+			)
+		)
+		(pin "DOUT" output
+			(at 63.5 172.72 0)
+			(effects
+				(font
+					(size 1.27 1.27)
+				)
+				(justify right)
+			)
+		)
+		(pin "LOAD" bidirectional
+			(at 63.5 162.56 0)
+			(effects
+				(font
+					(size 1.27 1.27)
+				)
+				(justify right)
+			)
+		)
+		(instances
+			(project "study focus device"
+				(path "/33a9b268-fa43-451b-98e7-c69879a56f92"
+					(page "8")
+				)
+			)
+		)
+	)
+	(sheet
+		(at 17.78 180.34)
+		(size 45.72 17.78)
+		(exclude_from_sim no)
+		(in_bom yes)
+		(on_board yes)
+		(dnp no)
+		(fields_autoplaced yes)
+		(stroke
+			(width 0.1524)
+			(type solid)
+		)
+		(fill
+			(color 0 0 0 0.0000)
+		)
+		(property "Sheetname" "LEDS2"
+			(at 17.78 179.6284 0)
+			(effects
+				(font
+					(size 1.27 1.27)
+				)
+				(justify left bottom)
+			)
+		)
+		(property "Sheetfile" "leds2.kicad_sch"
+			(at 17.78 198.7046 0)
+			(effects
+				(font
+					(size 1.27 1.27)
+				)
+				(justify left top)
+			)
+		)
+		(pin "CLK" bidirectional
+			(at 63.5 184.15 0)
+			(effects
+				(font
+					(size 1.27 1.27)
+				)
+				(justify right)
+			)
+		)
+		(pin "DIN" input
+			(at 63.5 181.61 0)
+			(effects
+				(font
+					(size 1.27 1.27)
+				)
+				(justify right)
+			)
+		)
+		(pin "LOAD" bidirectional
+			(at 63.5 186.69 0)
+			(effects
+				(font
+					(size 1.27 1.27)
+				)
+				(justify right)
+			)
+		)
+		(instances
+			(project "study focus device"
+				(path "/33a9b268-fa43-451b-98e7-c69879a56f92"
+					(page "9")
+				)
+			)

Commit message: more changes to the pcb
Other:
- added sheet Power module (power_module.kicad_sch)

Commit message: more work
Parts:
- added J1, J?: Conn_01x02_Pin, Connector_PinHeader_2.54mm:PinHeader_1x02_P2.54mm_Vertical, symbol Connector:Conn_01x02_Pin
- added J? (x2): Conn_01x03_Pin, Connector_PinHeader_2.54mm:PinHeader_1x03_P2.54mm_Vertical, symbol Connector:Conn_01x03_Pin
- added R? (x2): R, Resistor_THT:R_Axial_DIN0207_L6.3mm_D2.5mm_P7.62mm_Horizontal, symbol Device:R
Connections:
- net +3V3: now also J?.3 (Pin_3), R?.1, R?.1
- net CHIP SELECT: now also J?.3 (Pin_3)
- net CLK: now also J?.1 (Pin_1)
- net GND: now also J1.2 (Pin_2), J?.2 (Pin_2)
- net MOSI: now also J?.2 (Pin_2)
- net SCL: now also J?.2 (Pin_2), R?.2
- net SDA: now also J?.1 (Pin_1), R?.2
- new net +5V: J1.1 (Pin_1), J?.1 (Pin_1)
Other:
- removed sheet Power module
